File: SHS_DCDC/BAT.sch (KiCad schematic (older format))
At the start: 8 parts, among them Q10 PMV100XPEAR, Q11 PMV100XPEAR, Q12 PMV100XPEAR, Q9 PMV100XPEAR, U2 INA181

Commit message: esp32 s2 mini placed
Parts:
- 4cells1: footprint SHS_DCDC:BK-18650-PC8 -> BK-18650:BK-18650-PC8
- C6: symbol Device:C -> SHS_DCDC:C-Device
- R8: symbol Device:R -> SHS_DCDC:R-Device
- U2: symbol Amplifier_Current:INA181 -> SHS_DCDC:INA181-Amplifier_Current
Other:
- moved on the sheet: 4cells1, Q10, Q11, Q12, Q9
