File: SHS_DCDC/LOAD.sch (KiCad schematic (older format))
At the start: 49 parts, among them Q2 PMV100XPEAR, Q3 2N7002, Q4 2N7002, Q5 PMV100XPEAR, Q6 2N7002, Q7 PMV100XPEAR, U3 LMV324AIDR

Commit message: esp32 s2 mini placed
Parts:
- C10, C11, C12, C13, C14, C15, C16, C17, C18, C19, C7, C8, C9: symbol Device:C -> SHS_DCDC:C-Device
- Q3, Q4, Q6: symbol dk_Transistors-FETs-MOSFETs-Single:2N7002 -> SHS_DCDC:2N7002-dk_Transistors-FETs-MOSFETs-Single
- R10, R11, R12, R13, R14, R15, R16, R17, R18, R19, R20, R21, R22, R23, R24, R25, R26, R27, R28, R29, R30, R31, R32, R44, R45, R9: symbol Device:R -> SHS_DCDC:R-Device
- U3: symbol LMV324AIDR:LMV324AIDR -> SHS_DCDC:LMV324AIDR
