File: SHS_DCDC/MCU.sch (KiCad schematic (older format))
At the start: 7 parts, among them Q13 PMV100XPEAR, U6 STM32G050K8T6, U7 MCP101

Commit message: esp32 s2 mini placed
Parts:
- removed C30: 4.7uF, Capacitor_SMD:C_0603_1608Metric, symbol Device:C
- removed C31: 100nF, Capacitor_SMD:C_0402_1005Metric, symbol Device:C
- removed U6: STM32G050K8T6, SHS_DCDC:STM320G50_LQFP32, symbol SHS_DCDC:STM32G050K8T6
- added U6: ESP32-S2-MINI-1, Espressif:ESP32-S2-MINI-1, symbol Espressif:ESP32-S2-MINI-1
- C28, C29: symbol Device:C -> SHS_DCDC:C-Device
Connections:
- net labels added: GND-power
- net labels removed: GND
- wire segments 36 -> 35
Other:
- moved on the sheet: C28, C29, Q13, U7
