File: SHS_DCDC/USB.sch (KiCad schematic (older format))
At the start: 24 parts, among them J2 USB_A, Q8 Q_PMOS_DGS, U4 LMV358IDR, U5 MP3414A

Commit message: esp32 s2 mini placed
Parts:
- C20, C21, C22, C23, C24, C25, C26, C27: symbol Device:C -> SHS_DCDC:C-Device
- J2: symbol Connector:USB_A -> SHS_DCDC:USB_A-Connector
- L2: symbol Device:L -> SHS_DCDC:L-Device
- Q8: symbol Device:Q_PMOS_DGS -> SHS_DCDC:Q_PMOS_DGS-Device
- R33, R34, R35, R36, R37, R38, R39, R40, R41, R42, R43: symbol Device:R -> SHS_DCDC:R-Device
- U4: symbol dk_Linear-Amplifiers-Instrumentation-OP-Amps-Buffer-Amps:LMV358IDR -> SHS_DCDC:LMV358IDR-dk_Linear-Amplifiers-Instrumentation-OP-Amps-Buffer-Amps
Changed lines of the file:
@@
 $EndDescr
 $Comp
-L dk_Linear-Amplifiers-Instrumentation-OP-Amps-Buffer-Amps:LMV358IDR U4
+L SHS_DCDC:LMV358IDR-dk_Linear-Amplifiers-Instrumentation-OP-Amps-Buffer-Amps U4
 U 1 1 6085D38A
 P 5250 3900
@@
 $EndComp
 $Comp
-L dk_Linear-Amplifiers-Instrumentation-OP-Amps-Buffer-Amps:LMV358IDR U4
+L SHS_DCDC:LMV358IDR-dk_Linear-Amplifiers-Instrumentation-OP-Amps-Buffer-Amps U4
 U 2 1 6085E198
 P 8400 4050
@@
 	5250 4100 5250 4300
 $Comp
-L power:GND #PWR037
+L SHS_DCDC:GND-power #PWR037
 U 1 1 6086001C
 P 5250 4300
 F 0 "#PWR037" H 5250 4050 50  0001 C CNN
-F 1 "GND" H 5255 4127 50  0000 C CNN
+F 1 "GND-power" H 5255 4127 50  0000 C CNN
 F 2 "" H 5250 4300 50  0001 C CNN
 F 3 "" H 5250 4300 50  0001 C CNN
@@
 $EndComp
 $Comp
-L power:GND #PWR036
+L SHS_DCDC:GND-power #PWR036
 U 1 1 60860551
 P 7950 4050
 F 0 "#PWR036" H 7950 3800 50  0001 C CNN
-F 1 "GND" H 7955 3877 50  0000 C CNN
+F 1 "GND-power" H 7955 3877 50  0000 C CNN
 F 2 "" H 7950 4050 50  0001 C CNN
 F 3 "" H 7950 4050 50  0001 C CNN
@@
 I_USB
 $Comp
-L Device:C C20
+L SHS_DCDC:C-Device C20
 U 1 1 60864012
 P 5650 3450
@@
 	5800 3450 6000 3450
 $Comp
-L power:GND #PWR038
+L SHS_DCDC:GND-power #PWR038
 U 1 1 60864586
 P 6000 3450
 F 0 "#PWR038" H 6000 3200 50  0001 C CNN
-F 1 "GND" V 6005 3322 50  0000 R CNN
+F 1 "GND-power" V 6005 3322 50  0000 R CNN
 F 2 "" H 6000 3450 50  0001 C CNN
 F 3 "" H 6000 3450 50  0001 C CNN
@@
 	5550 3900 6100 3900
 $Comp
-L Device:R R40
+L SHS_DCDC:R-Device R40
 U 1 1 6086567E
 P 6250 3900
@@
 	5250 2500 5250 2850
 $Comp
-L Device:Q_PMOS_DGS Q8
+L SHS_DCDC:Q_PMOS_DGS-Device Q8
 U 1 1 6086A0AF
 P 6850 2950
@@
 Connection ~ 6850 3900
 $Comp
-L Device:C C21
+L SHS_DCDC:C-Device C21
 U 1 1 6086C143
 P 6850 4300
@@
 	6850 4450 6850 4600
 $Comp
-L power:GND #PWR039
+L SHS_DCDC:GND-power #PWR039
 U 1 1 6086CB94
 P 6850 4600
 F 0 "#PWR039" H 6850 4350 50  0001 C CNN
-F 1 "GND" H 6855 4427 50  0000 C CNN
+F 1 "GND-power" H 6855 4427 50  0000 C CNN
 F 2 "" H 6850 4600 50  0001 C CNN
 F 3 "" H 6850 4600 50  0001 C CNN
@@
 	7550 2850 7550 3050
 $Comp
-L Device:R R35
+L SHS_DCDC:R-Device R35
 U 1 1 60873238
 P 8400 2850
@@
 $EndComp
 $Comp
-L Device:R R33
+L SHS_DCDC:R-Device R33
 U 1 1 60874AF4
 P 7550 3200
@@
 $EndComp
 $Comp
-L Device:R R36
+L SHS_DCDC:R-Device R36
 U 1 1 608751B6
 P 9300 3200
@@
 Connection ~ 7550 3550
 $Comp
-L Device:R R34
+L SHS_DCDC:R-Device R34
 U 1 1 6087898E
 P 7550 4350
@@
 $EndComp
 $Comp
-L power:GND #PWR040
+L SHS_DCDC:GND-power #PWR040
 U 1 1 608792CF
 P 7550 5000
 F 0 "#PWR040" H 7550 4750 50  0001 C CNN
-F 1 "GND" H 7555 4827 50  0000 C CNN
+F 1 "GND-power" H 7555 4827 50  0000 C CNN
 F 2 "" H 7550 5000 50  0001 C CNN
 F 3 "" H 7550 5000 50  0001 C CNN
@@
 Connection ~ 9300 3550
 $Comp
-L Device:R R37
+L SHS_DCDC:R-Device R37
 U 1 1 60879A6C
 P 9300 4350
@@
 Connection ~ 9300 4700
 $Comp
-L Device:R R38
+L SHS_DCDC:R-Device R38
 U 1 1 6087C543
 P 9300 5100
@@
 	9300 5250 9300 5400
 $Comp
-L power:GND #PWR041
+L SHS_DCDC:GND-power #PWR041
 U 1 1 6087CE1B
 P 9300 5400
 F 0 "#PWR041" H 9300 5150 50  0001 C CNN
-F 1 "GND" H 9305 5227 50  0000 C CNN
+F 1 "GND-power" H 9305 5227 50  0000 C CNN
 F 2 "" H 9300 5400 50  0001 C CNN
 F 3 "" H 9300 5400 50  0001 C CNN
@@
 ILIM_USB
 $Comp
-L Device:R R?
+L SHS_DCDC:R-Device R?
 U 1 1 608940EB
 P 3450 3800
@@
 $EndComp
 $Comp
-L Device:C C?
+L SHS_DCDC:C-Device C?
 U 1 1 608940F1
 P 3900 4100
@@
 	3900 4250 3900 4400
 $Comp
-L power:GND #PWR?
+L SHS_DCDC:GND-power #PWR?
 U 1 1 608940FB
 P 3900 4400
@@
 AR Path="/6081F53E/608940FB" Ref="#PWR042"  Part="1"
 F 0 "#PWR042" H 3900 4150 50  0001 C CNN
-F 1 "GND" H 3905 4227 50  0000 C CNN
+F 1 "GND-power" H 3905 4227 50  0000 C CNN
 F 2 "" H 3900 4400 50  0001 C CNN
 F 3 "" H 3900 4400 50  0001 C CNN
@@
 	1300 2850 1300 3150
 $Comp
-L Device:C C23
+L SHS_DCDC:C-Device C23
 U 1 1 60AD32A1
 P 1300 3300
@@
 	1300 3450 1300 3700
 $Comp
-L power:GND #PWR043
+L SHS_DCDC:GND-power #PWR043
 U 1 1 60AD457F
 P 1300 3700
 F 0 "#PWR043" H 1300 3450 50  0001 C CNN
-F 1 "GND" H 1305 3527 50  0000 C CNN
+F 1 "GND-power" H 1305 3527 50  0000 C CNN
 F 2 "" H 1300 3700 50  0001 C CNN
 F 3 "" H 1300 3700 50  0001 C CNN
@@
 	2200 3400 2200 3600
 $Comp
-L power:GND #PWR044
+L SHS_DCDC:GND-power #PWR044
 U 1 1 60B04ECF
 P 2200 3600
 F 0 "#PWR044" H 2200 3350 50  0001 C CNN
-F 1 "GND" H 2205 3427 50  0000 C CNN
+F 1 "GND-power" H 2205 3427 50  0000 C CNN
 F 2 "" H 2200 3600 50  0001 C CNN
 F 3 "" H 2200 3600 50  0001 C CNN
@@
 $EndComp
 $Comp
-L power:GND #PWR045
+L SHS_DCDC:GND-power #PWR045
 U 1 1 60B056D9
 P 2350 3600
 F 0 "#PWR045" H 2350 3350 50  0001 C CNN
-F 1 "GND" H 2355 3427 50  0000 C CNN
+F 1 "GND-power" H 2355 3427 50  0000 C CNN
 F 2 "" H 2350 3600 50  0001 C CNN
 F 3 "" H 2350 3600 50  0001 C CNN
@@
 $EndComp
 $Comp
-L power:GND #PWR046
+L SHS_DCDC:GND-power #PWR046
 U 1 1 60B0589A
 P 2500 3600
 F 0 "#PWR046" H 2500 3350 50  0001 C CNN
-F 1 "GND" H 2505 3427 50  0000 C CNN
+F 1 "GND-power" H 2505 3427 50  0000 C CNN
 F 2 "" H 2500 3600 50  0001 C CNN
 F 3 "" H 2500 3600 50  0001 C CNN
@@
 	2500 3400 2500 3600
 $Comp
-L Device:L L2
+L SHS_DCDC:L-Device L2
 U 1 1 60B07CEE
 P 1650 2450
@@
 	2350 2450 2350 2550
 $Comp
-L Device:R R?
+L SHS_DCDC:R-Device R?
 U 1 1 60B0A4C6
 P 1750 3600
@@
 	5250 2850 3800 2850
 $Comp
-L Device:R R?
+L SHS_DCDC:R-Device R?
 U 1 1 60B12EAC
 P 3450 3150
@@
 	3300 3150 3000 3150
 $Comp
-L Device:R R?
+L SHS_DCDC:R-Device R?
 U 1 1 60B15A97
 P 3000 3400
@@
 	3150 3800 3300 3800
 $Comp
-L power:GND #PWR047
+L SHS_DCDC:GND-power #PWR047
 U 1 1 60B1AD2A
 P 3000 3650
 F 0 "#PWR047" H 3000 3400 50  0001 C CNN
-F 1 "GND" H 3005 3477 50  0000 C CNN
+F 1 "GND-power" H 3005 3477 50  0000 C CNN
 F 2 "" H 3000 3650 50  0001 C CNN
 F 3 "" H 3000 3650 50  0001 C CNN
@@
 Connection ~ 9300 2850
 $Comp
-L Connector:USB_A J2
+L SHS_DCDC:USB_A-Connector J2
 U 1 1 60B1D413
 P 9900 2650
@@
 	9900 1900 9650 1900
 $Comp
-L power:GND #PWR0106
+L SHS_DCDC:GND-power #PWR0106
 U 1 1 60B20271
 P 9650 1900
 F 0 "#PWR0106" H 9650 1650 50  0001 C CNN
-F 1 "GND" H 9655 1727 50  0000 C CNN
+F 1 "GND-power" H 9655 1727 50  0000 C CNN
 F 2 "" H 9650 1900 50  0001 C CNN
 F 3 "" H 9650 1900 50  0001 C CNN
@@
 	3100 2850 2800 2850
 $Comp
-L Device:C C24
+L SHS_DCDC:C-Device C24
 U 1 1 60B26581
 P 3100 2500
@@
 $EndComp
 $Comp
-L Device:C C25
+L SHS_DCDC:C-Device C25
 U 1 1 60B26A30
 P 3550 2500
@@
 	3100 2350 3100 2100
 $Comp
-L power:GND #PWR048
+L SHS_DCDC:GND-power #PWR048
 U 1 1 60B2BC8C
 P 3100 2100
 F 0 "#PWR048" H 3100 1850 50  0001 C CNN
-F 1 "GND" H 3105 1927 50  0000 C CNN
+F 1 "GND-power" H 3105 1927 50  0000 C CNN
 F 2 "" H 3100 2100 50  0001 C CNN
 F 3 "" H 3100 2100 50  0001 C CNN
@@
 $EndComp
 $Comp
-L power:GND #PWR049
+L SHS_DCDC:GND-power #PWR049
 U 1 1 60B2D929
 P 3550 2100
 F 0 "#PWR049" H 3550 1850 50  0001 C CNN
-F 1 "GND" H 3555 1927 50  0000 C CNN
+F 1 "GND-power" H 3555 1927 50  0000 C CNN
 F 2 "" H 3550 2100 50  0001 C CNN
 F 3 "" H 3550 2100 50  0001 C CNN
@@
 	6750 1950 6750 1700
 $Comp
-L Device:C C26
+L SHS_DCDC:C-Device C26
 U 1 1 60FFC505
 P 6750 1550
@@
 $EndComp
 $Comp
-L Device:C C27
+L SHS_DCDC:C-Device C27
 U 1 1 610067B7
 P 7550 1550
@@
 	7550 1400 7550 1150
 $Comp
-L power:GND #PWR0107
+L SHS_DCDC:GND-power #PWR0107
 U 1 1 6100D732
 P 6750 1150
 F 0 "#PWR0107" H 6750 900 50  0001 C CNN
-F 1 "GND" H 6755 977 50  0000 C CNN
+F 1 "GND-power" H 6755 977 50  0000 C CNN
 F 2 "" H 6750 1150 50  0001 C CNN
 F 3 "" H 6750 1150 50  0001 C CNN
@@
 $EndComp
 $Comp
-L power:GND #PWR0108
+L SHS_DCDC:GND-power #PWR0108
 U 1 1 610158D0
 P 7550 1150
 F 0 "#PWR0108" H 7550 900 50  0001 C CNN
-F 1 "GND" H 7555 977 50  0000 C CNN
+F 1 "GND-power" H 7555 977 50  0000 C CNN
 F 2 "" H 7550 1150 50  0001 C CNN
 F 3 "" H 7550 1150 50  0001 C CNN
