File: SHS_DCDC/MCU.kicad_sch (KiCad schematic)
At the start: 3 parts, among them Q13 PMV100XPEAR, U6 ESP32-S2-MINI-1

Commit message: Ubuntu transfer
Commit before transfer onto Ubuntu
Parts:
- added C28: 100nF, Capacitor_SMD:C_0402_1005Metric, symbol Device:C
- added C36: 1uF, Capacitor_SMD:C_0402_1005Metric, symbol Device:C
- added J3: Conn_ARM_JTAG_SWD_10, Connector_PinHeader_1.27mm:PinHeader_2x05_P1.27mm_Vertical, symbol Connector:Conn_ARM_JTAG_SWD_10
- added R21: 10k, Resistor_SMD:R_0402_1005Metric, symbol Device:R
- added S1: TS02-66-70-BK-160-LCR-D, SW_TS02-66-70-BK-160-LCR-D, symbol SHS_DCDC:TS02-66-70-BK-160-LCR-D
Connections:
- net GND: now also C28.2, C36.2, J3.3 (GND), J3.5 (GND), S1.3, S1.4
- net V_MCU: now also J3.1 (VTref), R21.1
- net USB_D-: now reaches U6.23 (USB_D-/ADC2_CH8/GPIO19)
- net USB_D+: now reaches U6.24 (USB_D+/ADC2_CH9/GPIO20)
- net MCU_MTCK: now reaches U6.35 (MTCK/JTAG/GPIO39)
- net MCU_MTCK: now also J3.4 (SWDCLK/TCK)
- net MCU_MTDO: now reaches U6.36 (MTDO/JTAG/GPIO40)
- net MCU_MTDO: now also J3.6 (SWO/TDO)
- net MCU_MTDI: now reaches U6.37 (MTDI/JTAG/GPIO41)
- net MCU_MTDI: now also J3.8 (NC/TDI)
- net MCU_MTMS: now reaches U6.38 (MTMS/JTAG/GPIO42)
- net MCU_MTMS: now also J3.2 (SWDIO/TMS)
- net MCU_RST: now reaches U6.45 (CHIP/PU/RESET)
- net MCU_RST: now also C28.1, C36.1, J3.10 (~{RESET}), R21.2, S1.1, S1.2
Other:
- note added: "Gives power to the MCU only after the battery is charged enough"
- moved on the sheet: Q13

Commit message: Commit_190223
Normal commit
Connections:
- net MCU_PWM_TL: now also U6.34 (GPIO38)
- net ODP_RESET: now reaches Q13.1 (G)
Other:
- moved on the sheet: J3
Changed lines of the file:
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@@
     (stroke (width 0) (type default) (color 0 0 0 0))
   )
-  (wire (pts (xy 232.41 88.9) (xy 241.3 88.9))
+  (wire (pts (xy 259.08 38.1) (xy 267.97 38.1))
     (stroke (width 0) (type default) (color 0 0 0 0))
   )
@@
     (stroke (width 0) (type default) (color 0 0 0 0))
   )
-  (wire (pts (xy 232.41 91.44) (xy 241.3 91.44))
-    (stroke (width 0) (type default) (color 0 0 0 0))
-  )
-  (wire (pts (xy 219.71 73.66) (xy 224.79 73.66))
+  (wire (pts (xy 259.08 40.64) (xy 267.97 40.64))
+    (stroke (width 0) (type default) (color 0 0 0 0))
+  )
+  (wire (pts (xy 246.38 22.86) (xy 251.46 22.86))
     (stroke (width 0) (type default) (color 0 0 0 0))
   )
@@
     (stroke (width 0) (type default) (color 0 0 0 0))
   )
-  (wire (pts (xy 232.41 96.52) (xy 241.3 96.52))
-    (stroke (width 0) (type default) (color 0 0 0 0))
-  )
-  (wire (pts (xy 232.41 93.98) (xy 241.3 93.98))
+  (wire (pts (xy 259.08 45.72) (xy 267.97 45.72))
+    (stroke (width 0) (type default) (color 0 0 0 0))
+  )
+  (wire (pts (xy 259.08 43.18) (xy 267.97 43.18))
     (stroke (width 0) (type default) (color 0 0 0 0))
   )
@@
     (stroke (width 0) (type default) (color 0 0 0 0))
   )
-  (wire (pts (xy 219.71 76.2) (xy 219.71 73.66))
+  (wire (pts (xy 246.38 25.4) (xy 246.38 22.86))
     (stroke (width 0) (type default) (color 0 0 0 0))
   )
@@
     (stroke (width 0) (type default) (color 0 0 0 0))
   )
+  (wire (pts (xy 179.07 87.63) (xy 187.96 87.63))
+    (stroke (width 0) (type default) (color 0 0 0 0))
+  )
   (wire (pts (xy 99.06 74.93) (xy 99.06 80.01))
     (stroke (width 0) (type default) (color 0 0 0 0))
@@
     (stroke (width 0) (type default) (color 0 0 0 0))
   )
-  (wire (pts (xy 219.71 106.68) (xy 219.71 113.03))
+  (wire (pts (xy 246.38 55.88) (xy 246.38 62.23))
     (stroke (width 0) (type default) (color 0 0 0 0))
   )
@@
     (stroke (width 0) (type default) (color 0 0 0 0))
   )
-  (wire (pts (xy 232.41 83.82) (xy 241.3 83.82))
+  (wire (pts (xy 259.08 33.02) (xy 267.97 33.02))
     (stroke (width 0) (type default) (color 0 0 0 0))
   )
@@
     )
   )
+  (global_label "ODP_RESET" (shape input) (at 59.69 58.42 270) (fields_autoplaced)
+    (effects (font (size 1.27 1.27)) (justify right))
+    (property "Intersheet References" "${INTERSHEET_REFS}" (id 0) (at 59.6106 71.3275 90)
+      (effects (font (size 1.27 1.27)) (justify right) hide)
+    )
+  )
   (global_label "USB_D+" (shape input) (at 190.5 120.65 0) (fields_autoplaced)
     (effects (font (size 1.27 1.27)) (justify left))
@@
     )
   )
-  (global_label "MCU_MTMS" (shape input) (at 241.3 91.44 0) (fields_autoplaced)
-    (effects (font (size 1.27 1.27)) (justify left))
-    (property "Intersheet References" "${INTERSHEET_REFS}" (id 0) (at 253.7237 91.3606 0)
-      (effects (font (size 1.27 1.27)) (justify left) hide)
-    )
-  )
-  (global_label "V_MCU" (shape input) (at 224.79 73.66 0) (fields_autoplaced)
-    (effects (font (size 1.27 1.27)) (justify left))
-    (property "Intersheet References" "${INTERSHEET_REFS}" (id 0) (at 233.2223 73.5806 0)
-      (effects (font (size 1.27 1.27)) (justify left) hide)
-    )
-  )
-  (global_label "MCU_MTCK" (shape input) (at 241.3 88.9 0) (fields_autoplaced)
-    (effects (font (size 1.27 1.27)) (justify left))
-    (property "Intersheet References" "${INTERSHEET_REFS}" (id 0) (at 253.6028 88.8206 0)
+  (global_label "MCU_MTMS" (shape input) (at 267.97 40.64 0) (fields_autoplaced)
+    (effects (font (size 1.27 1.27)) (justify left))
+    (property "Intersheet References" "${INTERSHEET_REFS}" (id 0) (at 280.3937 40.5606 0)
+      (effects (font (size 1.27 1.27)) (justify left) hide)
+    )
+  )
+  (global_label "V_MCU" (shape input) (at 251.46 22.86 0) (fields_autoplaced)
+    (effects (font (size 1.27 1.27)) (justify left))
+    (property "Intersheet References" "${INTERSHEET_REFS}" (id 0) (at 259.8923 22.7806 0)
+      (effects (font (size 1.27 1.27)) (justify left) hide)
+    )
+  )
+  (global_label "MCU_MTCK" (shape input) (at 267.97 38.1 0) (fields_autoplaced)
+    (effects (font (size 1.27 1.27)) (justify left))
+    (property "Intersheet References" "${INTERSHEET_REFS}" (id 0) (at 280.2728 38.0206 0)
       (effects (font (size 1.27 1.27)) (justify left) hide)
     )
@@
     )
   )
-  (global_label "MCU_RST" (shape input) (at 241.3 83.82 0) (fields_autoplaced)
-    (effects (font (size 1.27 1.27)) (justify left))
-    (property "Intersheet References" "${INTERSHEET_REFS}" (id 0) (at 252.0909 83.7406 0)
+  (global_label "MCU_RST" (shape input) (at 267.97 33.02 0) (fields_autoplaced)
+    (effects (font (size 1.27 1.27)) (justify left))
+    (property "Intersheet References" "${INTERSHEET_REFS}" (id 0) (at 278.7609 32.9406 0)
       (effects (font (size 1.27 1.27)) (justify left) hide)
     )
@@
     )
   )
-  (global_label "MCU_MTDO" (shape input) (at 241.3 93.98 0) (fields_autoplaced)
-    (effects (font (size 1.27 1.27)) (justify left))
-    (property "Intersheet References" "${INTERSHEET_REFS}" (id 0) (at 253.6632 93.9006 0)
+  (global_label "MCU_MTDO" (shape input) (at 267.97 43.18 0) (fields_autoplaced)
+    (effects (font (size 1.27 1.27)) (justify left))
+    (property "Intersheet References" "${INTERSHEET_REFS}" (id 0) (at 280.3332 43.1006 0)
       (effects (font (size 1.27 1.27)) (justify left) hide)
     )
@@
     )
   )
-  (global_label "MCU_MTDI" (shape input) (at 241.3 96.52 0) (fields_autoplaced)
-    (effects (font (size 1.27 1.27)) (justify left))
-    (property "Intersheet References" "${INTERSHEET_REFS}" (id 0) (at 252.9375 96.4406 0)
+  (global_label "MCU_PWM_TL" (shape input) (at 187.96 87.63 0) (fields_autoplaced)
+    (effects (font (size 1.27 1.27)) (justify left))
+    (property "Intersheet References" "${INTERSHEET_REFS}" (id 0) (at 202.4399 87.5506 0)
+      (effects (font (size 1.27 1.27)) (justify left) hide)
+    )
+  )
+  (global_label "MCU_MTDI" (shape input) (at 267.97 45.72 0) (fields_autoplaced)
+    (effects (font (size 1.27 1.27)) (justify left))
+    (property "Intersheet References" "${INTERSHEET_REFS}" (id 0) (at 279.6075 45.6406 0)
       (effects (font (size 1.27 1.27)) (justify left) hide)
     )
@@
     (pin "1")
   )
-  (symbol (lib_id "SHS_DCDC:GND-power") (at 219.71 113.03 0) (unit 1)
-    (in_bom yes) (on_board yes)
-    (property "Reference" "#PWR0110" (id 0) (at 219.71 119.38 0)
-      (effects (font (size 1.27 1.27)) hide)
-    )
-    (property "Value" "GND-power" (id 1) (at 219.837 116.2812 90)
-      (effects (font (size 1.27 1.27)) (justify right))
-    )
-    (property "Footprint" "" (id 2) (at 219.71 113.03 0)
-      (effects (font (size 1.27 1.27)) hide)
-    )
-    (property "Datasheet" "" (id 3) (at 219.71 113.03 0)
-      (effects (font (size 1.27 1.27)) hide)
-    )
-    (pin "1")
-  )
-  (symbol (lib_id "Connector:Conn_ARM_JTAG_SWD_10") (at 219.71 91.44 0) (unit 1)
+  (symbol (lib_id "SHS_DCDC:GND-power") (at 246.38 62.23 0) (unit 1)
+    (in_bom yes) (on_board yes)
+    (property "Reference" "#PWR0110" (id 0) (at 246.38 68.58 0)
+      (effects (font (size 1.27 1.27)) hide)
+    )
+    (property "Value" "GND-power" (id 1) (at 246.507 65.4812 90)
+      (effects (font (size 1.27 1.27)) (justify right))
+    )
+    (property "Footprint" "" (id 2) (at 246.38 62.23 0)
+      (effects (font (size 1.27 1.27)) hide)
+    )
+    (property "Datasheet" "" (id 3) (at 246.38 62.23 0)
+      (effects (font (size 1.27 1.27)) hide)
+    )
+    (pin "1")
+  )
+  (symbol (lib_id "Connector:Conn_ARM_JTAG_SWD_10") (at 246.38 40.64 0) (unit 1)
     (in_bom yes) (on_board yes) (fields_autoplaced)
-    (property "Reference" "J3" (id 0) (at 208.28 90.1699 0)
-      (effects (font (size 1.27 1.27)) (justify right))
-    )
-    (property "Value" "Conn_ARM_JTAG_SWD_10" (id 1) (at 208.28 92.7099 0)
-      (effects (font (size 1.27 1.27)) (justify right))
-    )
-    (property "Footprint" "Connector_PinHeader_1.27mm:PinHeader_2x05_P1.27mm_Vertical" (id 2) (at 219.71 91.44 0)
-      (effects (font (size 1.27 1.27)) hide)
-    )
-    (property "Datasheet" "http://infocenter.arm.com/help/topic/com.arm.doc.ddi0314h/DDI0314H_coresight_components_trm.pdf" (id 3) (at 210.82 123.19 90)
-      (effects (font (size 1.27 1.27)) hide)
-    )
+    (property "Reference" "J3" (id 0) (at 234.95 39.3699 0)
+      (effects (font (size 1.27 1.27)) (justify right))
+    )
+    (property "Value" "Conn_ARM_JTAG_SWD_10" (id 1) (at 234.95 41.9099 0)
+      (effects (font (size 1.27 1.27)) (justify right))
+    )
+    (property "Footprint" "Connector_PinHeader_1.27mm:PinHeader_2x05_P1.27mm_Vertical" (id 2) (at 246.38 40.64 0)
+      (effects (font (size 1.27 1.27)) hide)
+    )
+    (property "Datasheet" "http://infocenter.arm.com/help/topic/com.arm.doc.ddi0314h/DDI0314H_coresight_components_trm.pdf" (id 3) (at 237.49 72.39 90)
+      (effects (font (size 1.27 1.27)) hide)
+    )

Commit message: Commit_Fix
Fix to move back to ESP32
Connections:
- net MCU_PWM_BL1: now also U6.33 (GPIO37)
- net MCU_PWM_BL2: now also U6.32 (GPIO36)
- net MCU_PWM_MPPT: now also U6.29 (GPIO34)
Other:
- moved on the sheet: U6

Commit message: ProgressMisc
Parts:
- added C2, C37: TBD, Capacitor_SMD:C_0402_1005Metric, symbol Device:C
- added Y1: 2-SMD no lead, Crystal:Crystal_SMD_3215-2Pin_3.2x1.5mm, symbol Device:Crystal
Connections:
- net GND: now also C2.2, C37.2
- net at U6.19 (GPIO15/ADC2_CH4/XTAL_32K_P): now also C2.1, Y1.2
- net at U6.20 (GPIO16/ADC2_CH5/XTAL_32K_N): now also C37.1, Y1.1
Other:
- moved on the sheet: C29

Commit message: OCP
Adding overcharge protection
Parts:
- removed Q13: PMV100XPEAR, digikey-footprints:SOT-23-3, symbol SHS_DCDC:PMV100XPEAR
- added C39: 10uF, Capacitor_SMD:C_0805_2012Metric, symbol Device:C
- added C40: 1uF, Capacitor_SMD:C_0603_1608Metric, symbol Device:C
- added U8: MIC5501-3.0YM5, Package_TO_SOT_SMD:SOT-23-5, symbol Regulator_Linear:MIC5501-3.0YM5
Connections:
- net GND: now also C39.1, C40.2, U8.2 (GND)
- net LOAD: now also C39.2, U8.1 (VIN)
- net MCU_BL2_ONOFFSIG: now also U6.26 (SPI_CS1/GPIO26)
- net ODP_RESET: now also U8.3 (EN)
- net V_MCU: now also C40.1, U8.5 (VOUT)
- net MCU_OCP_BAT: now reaches U6.5 (GPIO1/ADC1_CH0)
Other:
- moved on the sheet: C36, U6

Commit message: 6 layers PCB
Decision to move to a 6 layers PCB to ease the PCB routing
Connections:
- net MCU_BL1_ONOFFSIG: now also U6.26 (SPI_CS1/GPIO26)
- net MCU_BL2_ONOFFSIG: now also U6.25 (GPIO21); no longer U6.26 (SPI_CS1/GPIO26)
- net MCU_MPPT_ENABLE: now also U6.31 (GPIO35)
- net MCU_TL_ONOFFSIG: now also U6.44 (GPIO46)
- net MCU_5V_EN: now reaches U6.17 (GPIO13/ADC2_CH2)
Changed lines of the file:
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@@
     (stroke (width 0) (type default) (color 0 0 0 0))
   )
-  (wire (pts (xy -87.63 72.39) (xy -73.66 72.39))
-    (stroke (width 0) (type default) (color 0 0 0 0))
-  )
-  (wire (pts (xy -38.1 73.66) (xy -27.94 73.66))
+  (wire (pts (xy 215.9 95.25) (xy 228.6 95.25))
+    (stroke (width 0) (type default) (color 0 0 0 0))
+  )
+  (wire (pts (xy 228.6 115.57) (xy 215.9 115.57))
     (stroke (width 0) (type default) (color 0 0 0 0))
   )
@@
     (stroke (width 0) (type default) (color 0 0 0 0))
   )
-  (wire (pts (xy -91.44 87.63) (xy -73.66 87.63))
+  (wire (pts (xy 132.08 118.11) (xy 143.51 118.11))
     (stroke (width 0) (type default) (color 0 0 0 0))
   )
@@
     (stroke (width 0) (type default) (color 0 0 0 0))
   )
-  (wire (pts (xy 224.79 92.71) (xy 215.9 92.71))
+  (wire (pts (xy 228.6 92.71) (xy 215.9 92.71))
     (stroke (width 0) (type default) (color 0 0 0 0))
   )
@@
     (stroke (width 0) (type default) (color 0 0 0 0))
   )
-  (wire (pts (xy -88.9 46.99) (xy -73.66 46.99))
+  (wire (pts (xy 228.6 105.41) (xy 215.9 105.41))
     (stroke (width 0) (type default) (color 0 0 0 0))
   )
@@
     (stroke (width 0) (type default) (color 0 0 0 0))
   )
-  (wire (pts (xy 233.68 97.79) (xy 215.9 97.79))
+  (wire (pts (xy 228.6 97.79) (xy 215.9 97.79))
     (stroke (width 0) (type default) (color 0 0 0 0))
   )
@@
     (stroke (width 0) (type default) (color 0 0 0 0))
   )
-  (wire (pts (xy 224.79 90.17) (xy 215.9 90.17))
+  (wire (pts (xy 228.6 90.17) (xy 215.9 90.17))
     (stroke (width 0) (type default) (color 0 0 0 0))
   )
@@
     (stroke (width 0) (type default) (color 0 0 0 0))
   )
-  (wire (pts (xy 231.14 113.03) (xy 215.9 113.03))
+  (wire (pts (xy 228.6 113.03) (xy 215.9 113.03))
     (stroke (width 0) (type default) (color 0 0 0 0))
   )
@@
     (stroke (width 0) (type default) (color 0 0 0 0))
   )
-  (wire (pts (xy 215.9 87.63) (xy 224.79 87.63))
+  (wire (pts (xy 215.9 87.63) (xy 228.6 87.63))
     (stroke (width 0) (type default) (color 0 0 0 0))
   )
@@
     (stroke (width 0) (type default) (color 0 0 0 0))
   )
-  (wire (pts (xy 125.73 87.63) (xy 143.51 87.63))
+  (wire (pts (xy 132.08 87.63) (xy 143.51 87.63))
     (stroke (width 0) (type default) (color 0 0 0 0))
   )
@@
     )
   )
-  (global_label "MCU_MPPT_ENABLE" (shape input) (at -87.63 72.39 180) (fields_autoplaced)
-    (effects (font (size 1.27 1.27)) (justify right))
-    (property "Intersheet References" "${INTERSHEET_REFS}" (id 0) (at 0 0 0)
+  (global_label "MCU_MPPT_ENABLE" (shape input) (at 228.6 95.25 0) (fields_autoplaced)
+    (effects (font (size 1.27 1.27)) (justify left))
+    (property "Intersheet References" "${INTERSHEET_REFS}" (id 0) (at 140.97 167.64 0)
       (effects (font (size 1.27 1.27)) hide)
     )
@@
     )
   )
-  (global_label "MCU_5V_ONOFF" (shape input) (at -91.44 87.63 180) (fields_autoplaced)
-    (effects (font (size 1.27 1.27)) (justify right))
-    (property "Intersheet References" "${INTERSHEET_REFS}" (id 0) (at 0 0 0)
-      (effects (font (size 1.27 1.27)) hide)
-    )
-  )
-  (global_label "MCU_PWM_MPPT" (shape input) (at 233.68 97.79 0) (fields_autoplaced)
-    (effects (font (size 1.27 1.27)) (justify left))
-    (property "Intersheet References" "${INTERSHEET_REFS}" (id 0) (at 185.42 144.78 0)
+  (global_label "MCU_5V_EN" (shape input) (at 132.08 118.11 180) (fields_autoplaced)
+    (effects (font (size 1.27 1.27)) (justify right))
+    (property "Intersheet References" "${INTERSHEET_REFS}" (id 0) (at 118.991 118.0306 0)
+      (effects (font (size 1.27 1.27)) (justify right) hide)
+    )
+  )
+  (global_label "MCU_PWM_MPPT" (shape input) (at 228.6 97.79 0) (fields_autoplaced)
+    (effects (font (size 1.27 1.27)) (justify left))
+    (property "Intersheet References" "${INTERSHEET_REFS}" (id 0) (at 180.34 144.78 0)
       (effects (font (size 1.27 1.27)) hide)
     )
@@
     )
   )
-  (global_label "MCU_PWM_BL2" (shape input) (at 224.79 92.71 0) (fields_autoplaced)
-    (effects (font (size 1.27 1.27)) (justify left))
-    (property "Intersheet References" "${INTERSHEET_REFS}" (id 0) (at 175.26 161.29 0)
+  (global_label "MCU_PWM_BL2" (shape input) (at 228.6 92.71 0) (fields_autoplaced)
+    (effects (font (size 1.27 1.27)) (justify left))
+    (property "Intersheet References" "${INTERSHEET_REFS}" (id 0) (at 179.07 161.29 0)
       (effects (font (size 1.27 1.27)) hide)
     )
@@
     )
   )
-  (global_label "MCU_BL1_ONOFFSIG" (shape input) (at -38.1 73.66 180) (fields_autoplaced)
-    (effects (font (size 1.27 1.27)) (justify right))
-    (property "Intersheet References" "${INTERSHEET_REFS}" (id 0) (at 50.8 17.78 0)
+  (global_label "MCU_BL1_ONOFFSIG" (shape input) (at 228.6 113.03 0) (fields_autoplaced)
+    (effects (font (size 1.27 1.27)) (justify left))
+    (property "Intersheet References" "${INTERSHEET_REFS}" (id 0) (at 139.7 168.91 0)
       (effects (font (size 1.27 1.27)) hide)
     )
@@
     )
   )
-  (global_label "MCU_BL2_ONOFFSIG" (shape input) (at 231.14 113.03 0) (fields_autoplaced)
-    (effects (font (size 1.27 1.27)) (justify left))
-    (property "Intersheet References" "${INTERSHEET_REFS}" (id 0) (at 142.24 176.53 0)
-      (effects (font (size 1.27 1.27)) hide)
-    )
-  )
-  (global_label "MCU_OCP_BAT" (shape input) (at 125.73 87.63 180) (fields_autoplaced)
-    (effects (font (size 1.27 1.27)) (justify right))
-    (property "Intersheet References" "${INTERSHEET_REFS}" (id 0) (at 110.222 87.5506 0)
+  (global_label "MCU_BL2_ONOFFSIG" (shape input) (at 228.6 115.57 0) (fields_autoplaced)
+    (effects (font (size 1.27 1.27)) (justify left))
+    (property "Intersheet References" "${INTERSHEET_REFS}" (id 0) (at 139.7 179.07 0)
+      (effects (font (size 1.27 1.27)) hide)
+    )
+  )
+  (global_label "MCU_OCP_BAT" (shape input) (at 132.08 87.63 180) (fields_autoplaced)
+    (effects (font (size 1.27 1.27)) (justify right))
+    (property "Intersheet References" "${INTERSHEET_REFS}" (id 0) (at 116.572 87.5506 0)
       (effects (font (size 1.27 1.27)) (justify right) hide)
     )
@@
     )
   )
-  (global_label "MCU_TL_ONOFFSIG" (shape input) (at -88.9 46.99 180) (fields_autoplaced)
-    (effects (font (size 1.27 1.27)) (justify right))
-    (property "Intersheet References" "${INTERSHEET_REFS}" (id 0) (at 0 0 0)
-      (effects (font (size 1.27 1.27)) hide)
-    )
-  )
-  (global_label "MCU_PWM_BL1" (shape input) (at 224.79 90.17 0) (fields_autoplaced)
-    (effects (font (size 1.27 1.27)) (justify left))
-    (property "Intersheet References" "${INTERSHEET_REFS}" (id 0) (at 175.26 151.13 0)
+  (global_label "MCU_TL_ONOFFSIG" (shape input) (at 228.6 105.41 0) (fields_autoplaced)
+    (effects (font (size 1.27 1.27)) (justify left))
+    (property "Intersheet References" "${INTERSHEET_REFS}" (id 0) (at 139.7 152.4 0)
+      (effects (font (size 1.27 1.27)) hide)
+    )
+  )
+  (global_label "MCU_PWM_BL1" (shape input) (at 228.6 90.17 0) (fields_autoplaced)
+    (effects (font (size 1.27 1.27)) (justify left))
+    (property "Intersheet References" "${INTERSHEET_REFS}" (id 0) (at 179.07 151.13 0)
       (effects (font (size 1.27 1.27)) hide)
     )
@@
     )
   )
-  (global_label "MCU_PWM_TL" (shape input) (at 224.79 87.63 0) (fields_autoplaced)
-    (effects (font (size 1.27 1.27)) (justify left))
-    (property "Intersheet References" "${INTERSHEET_REFS}" (id 0) (at 239.2699 87.5506 0)
-      (effects (font (size 1.27 1.27)) (justify left) hide)
-    )
+  (global_label "MCU_PWM_TL" (shape input) (at 228.6 87.63 0) (fields_autoplaced)
+    (effects (font (size 1.27 1.27)) (justify left))
+    (property "Intersheet References" "${INTERSHEET_REFS}" (id 0) (at 243.0799 87.5506 0)
+      (effects (font (size 1.27 1.27)) (justify left) hide)
+    )
