File: SHS_DCDC/USB.kicad_sch (KiCad schematic)
At the start: 26 parts, among them J2 USB_A, Q8 Q_PMOS_DGS, U4 LMV358IDR, U5 MP3414A

Commit message: 3D rendering progress
Parts:
- L2: value L -> 1.5 uH; Ref (none) -> NR6028T1R5N
Changed lines of the file:
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@@
     (in_bom yes) (on_board yes)
     (property "Reference" "L2" (id 0) (at 41.91 57.6326 90))
-    (property "Value" "L" (id 1) (at 41.91 59.944 90))
+    (property "Value" "1.5 uH" (id 1) (at 41.91 59.944 90))
     (property "Footprint" "Inductor_SMD:L_Taiyo-Yuden_NR-60xx" (id 2) (at 41.91 62.23 0)
       (effects (font (size 1.27 1.27)) hide)
@@
       (effects (font (size 1.27 1.27)) hide)
     )
+    (property "Ref" "NR6028T1R5N" (id 4) (at 41.91 62.23 90)
+      (effects (font (size 1.27 1.27)) hide)
+    )

Commit message: PV input Power
Big modification on the PV input power protection, precisely on the reverse battery current protection, and also on the switch between direct PV charging and the DCDC converter
Parts:
- removed Q8: Q_PMOS_DGS, digikey-footprints:SOT-23-3, symbol SHS_DCDC:Q_PMOS_DGS-Device
- added Q8: PMV100XPEAR, digikey-kicad-library-master:SOT-23-3, symbol SHS_DCDC:PMV100XPEAR
- C20: footprint Capacitor_SMD:C_0603_1608Metric -> Capacitor_SMD:C_0402_1005Metric
Connections:
- net USB_OUT is gone; now on net 5V: U4.8 (VCC+)
- net 5V: now also Q8.2 (S)
- net at C21.2, R40.1: now also Q8.1 (G)
- net at R33.2, R35.2: now also Q8.3 (D)
- net I_USB renamed MCU_I_USB
Changed lines of the file:
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@@
     (stroke (width 0) (type default) (color 0 0 0 0))
   )
-  (wire (pts (xy 139.7 72.39) (xy 168.91 72.39))
+  (wire (pts (xy 139.7 72.39) (xy 171.45 72.39))
     (stroke (width 0) (type default) (color 0 0 0 0))
   )
@@
     (stroke (width 0) (type default) (color 0 0 0 0))
   )
-  (wire (pts (xy 179.07 72.39) (xy 191.77 72.39))
+  (wire (pts (xy 181.61 72.39) (xy 191.77 72.39))
     (stroke (width 0) (type default) (color 0 0 0 0))
   )
@@
     (stroke (width 0) (type default) (color 0 0 0 0))
   )
-  (wire (pts (xy 132.08 123.19) (xy 128.27 123.19))
+  (wire (pts (xy 132.08 123.19) (xy 129.54 123.19))
     (stroke (width 0) (type default) (color 0 0 0 0))
   )
@@
     (stroke (width 0) (type default) (color 0 0 0 0))
   )
-  (wire (pts (xy 173.99 120.65) (xy 173.99 80.01))
+  (wire (pts (xy 173.99 120.65) (xy 173.99 81.28))
     (stroke (width 0) (type default) (color 0 0 0 0))
   )
@@
     (stroke (width 0) (type default) (color 0 0 0 0))
   )
-  (text "Work principle of the USB current limit:\na shunt resistor create a drop dV.\nThat drop is amplified a 100 times.\nThat voltage called V(I_USB) is compared to a reference voltage called V(ILIM_USB).\nThat ILIM_USB value gives the limit of current according to:\nI = V(ILIM_USB)/(100 x R)\nThat means if you select V(ILIM_USB)=1V and R = 10 mOhm then I = 1 A\n* we call it actually MCU_ILIM_USB because that voltage is controlled by the ESP32\nExtra note: by default V(ILIM_USB) is 1V according to the voltage divider (in case the MCU is faulty)"
+  (text "Work principle of the USB current limit:\na shunt resistor create a drop dV.\nThat drop is amplified a 100 times.\nThat voltage called V(I_USB) is compared to a reference voltage called V(ILIM_USB).\nThat ILIM_USB value gives the limit of current according to:\nI = V(ILIM_USB)/(100 x R)\nThat means if you select V(ILIM_USB)=1V and R = 10 mOhm then I = 1 A\n* we call it actually MCU_ILIM_USB because that voltage is controlled by the ESP32\nNote: by default V(ILIM_USB) is 1V according to the voltage divider (in case the MCU is faulty)\nExtra note! we can read the current really going out, through the reading of MCU_USB_I"
     (at 113.03 35.56 0)
     (effects (font (size 1.27 1.27)) (justify left bottom))
   )
-  (global_label "USB_OUT" (shape input) (at 224.79 102.87 0) (fields_autoplaced)
+  (global_label "5V" (shape input) (at 224.79 102.87 0) (fields_autoplaced)
     (effects (font (size 1.27 1.27)) (justify left))
-    (property "Intersheet References" "${INTERSHEET_REFS}" (id 0) (at 0 0 0)
-      (effects (font (size 1.27 1.27)) hide)
+    (property "Intersheet References" "${INTERSHEET_REFS}" (id 0) (at 229.4123 102.7906 0)
+      (effects (font (size 1.27 1.27)) (justify left) hide)
     )
   )
@@
     )
   )
-  (global_label "I_USB" (shape input) (at 213.36 129.54 270) (fields_autoplaced)
+  (global_label "MCU_I_USB" (shape input) (at 213.36 129.54 270) (fields_autoplaced)
     (effects (font (size 1.27 1.27)) (justify right))
-    (property "Intersheet References" "${INTERSHEET_REFS}" (id 0) (at 0 0 0)
-      (effects (font (size 1.27 1.27)) hide)
+    (property "Intersheet References" "${INTERSHEET_REFS}" (id 0) (at 213.2806 142.2661 90)
+      (effects (font (size 1.27 1.27)) (justify right) hide)
     )
   )
@@
     )
   )
-  (global_label "I_USB" (shape input) (at 128.27 123.19 180) (fields_autoplaced)
+  (global_label "MCU_I_USB" (shape input) (at 129.54 123.19 180) (fields_autoplaced)
     (effects (font (size 1.27 1.27)) (justify right))
-    (property "Intersheet References" "${INTERSHEET_REFS}" (id 0) (at 10.16 21.59 0)
-      (effects (font (size 1.27 1.27)) hide)
+    (property "Intersheet References" "${INTERSHEET_REFS}" (id 0) (at 116.8139 123.1106 0)
+      (effects (font (size 1.27 1.27)) (justify right) hide)
     )
   )
@@
     (property "Reference" "C20" (id 0) (at 149.86 102.8192 90))
     (property "Value" "100nF" (id 1) (at 149.86 105.1306 90))
-    (property "Footprint" "Capacitor_SMD:C_0603_1608Metric" (id 2) (at 146.05 110.1852 0)
+    (property "Footprint" "Capacitor_SMD:C_0402_1005Metric" (id 2) (at 146.05 110.1852 0)
       (effects (font (size 1.27 1.27)) hide)
     )
@@
     (pin "1")
     (pin "2")
-  )
-  (symbol (lib_id "SHS_DCDC:Q_PMOS_DGS-Device") (at 173.99 74.93 270) (mirror x) (unit 1)
-    (in_bom yes) (on_board yes)
-    (property "Reference" "Q8" (id 0) (at 173.99 66.2432 90))
-    (property "Value" "Q_PMOS_DGS" (id 1) (at 173.99 68.5546 90))
-    (property "Footprint" "digikey-footprints:SOT-23-3" (id 2) (at 176.53 69.85 0)
-      (effects (font (size 1.27 1.27)) hide)
-    )
-    (property "Datasheet" "~" (id 3) (at 173.99 74.93 0)
-      (effects (font (size 1.27 1.27)) hide)
-    )
-    (pin "1")
-    (pin "2")
-    (pin "3")
   )
   (symbol (lib_id "SHS_DCDC:C-Device") (at 173.99 130.81 180) (unit 1)
@@
     (pin "2")
   )
+  (symbol (lib_id "SHS_DCDC:PMV100XPEAR") (at 176.53 72.39 270) (mirror x) (unit 1)
+    (in_bom yes) (on_board yes) (fields_autoplaced)
+    (property "Reference" "Q8" (id 0) (at 175.0703 64.77 90)
+      (effects (font (size 1.524 1.524)))
+    )
+    (property "Value" "PMV100XPEAR" (id 1) (at 175.0703 68.58 90)
+      (effects (font (size 1.524 1.524)))
+    )
+    (property "Footprint" "digikey-kicad-library-master:SOT-23-3" (id 2) (at 181.61 67.31 0)
+      (effects (font (size 1.524 1.524)) (justify left) hide)
+    )
+    (property "Datasheet" "" (id 3) (at 184.15 67.31 0)
+      (effects (font (size 1.524 1.524)) (justify left) hide)
+    )
+    (property "MPN" "PMV100XPEAR" (id 4) (at 189.23 67.31 0)
+      (effects (font (size 1.524 1.524)) (justify left) hide)
+    )
+    (property "Category" "Discrete Semiconductor Products" (id 5) (at 191.77 67.31 0)
+      (effects (font (size 1.524 1.524)) (justify left) hide)
+    )
+    (property "Family" "Transistors - FETs, MOSFETs - Single" (id 6) (at 194.31 67.31 0)
+      (effects (font (size 1.524 1.524)) (justify left) hide)
+    )
+    (property "Description" "MOSFET P-CH 20V 2.4A SOT23" (id 7) (at 196.85 67.31 0)
+      (effects (font (size 1.524 1.524)) (justify left) hide)
+    )
+    (property "Manufacturer" "Nexperia USA" (id 8) (at 199.39 67.31 0)
+      (effects (font (size 1.524 1.524)) (justify left) hide)
+    )
+    (property "Status" "Active" (id 9) (at 201.93 67.31 0)
+      (effects (font (size 1.524 1.524)) (justify left) hide)
+    )
+    (pin "1")
+    (pin "2")
+    (pin "3")
+  )
   (symbol (lib_id "SHS_DCDC:GND-power") (at 80.01 106.68 270) (unit 1)
