File: SHS_DCDC/USB.kicad_sch (KiCad schematic)
At the start: 26 parts, among them J2 USB_A, Q8 PMV100XPEAR, U4 LMV358IDR, U5 MP3414A

Commit message: Testpoints
All the tests points have been placed
Parts:
- removed R41: 100k, Resistor_SMD:R_0603_1608Metric, symbol SHS_DCDC:R-Device
- added C47: 1uF, Capacitor_SMD:C_0603_1608Metric, symbol SHS_DCDC:C-Device
- added D2: D_Schottky, Diode_SMD:D_SOD-523, symbol Device:D_Schottky
- added R65: 10k, Resistor_SMD:R_0603_1608Metric, symbol SHS_DCDC:R-Device
- added TP1, TP10, TP2, TP8: 5029, digikey-footprints:PC_Test_Point_Mini_3.8x2.03mm, symbol dk_Test-Points:5029
Connections:
- net 5V: now also TP2.1
- net GND: now also C47.2
- net USB_SHORT: now reaches C26.2, C27.2, J2.1 (VBUS), R35.1, R36.2
- net USB_SHORT: now also D2.1 (K)
- net at Q8.3 (D), R33.2, R35.2: now also TP8.1
- net MCU_5V_EN renamed MCU_USB_EN
- net MCU_USB_EN: now also C47.1, R65.2, TP10.1
- net MCU_ILIM_USB renamed MCU_USB_ILIM
- net MCU_USB_ILIM: now also TP1.1
- net MCU_I_USB renamed USB_I
- new net: D2.2 (A), R65.1
Other:
- note added: "Shunt resistor"
- note added: "Work principle of the USB current limit: a shunt resistor create a drop dV. That drop is amplified a 100 times. That voltage called V(I_USB) is compared to a reference voltage called V(ILIM_USB). That ILIM_USB value gives the limit of current according to: I = V(ILIM_USB)/(100 x R) That means if you select V(ILIM_USB)=1V and R = 10 mOhm then I = 1 A The ILIM_USB signal is connected to the DAC of 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"
- note added: "Work principle of the USB shortcut detection: The enable line is first activated, with a value high. This charge a capacitor. We then put the MCU_USB_EN to high Z for a time T. During that time T, if there is no shortcut, that capacitor leaks into the high Z of the EN line and MCU GPIO. Therefore, its voltage should be maintained high enough to let the DCDC converter ON. At the end of this time T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"
- note removed: "Work principle of the USB current limit: a shunt resistor create a drop dV. That drop is amplified a 100 times. That voltage called V(I_USB) is compared to a reference voltage called V(ILIM_USB). That ILIM_USB value gives the limit of current according to: I = V(ILIM_USB)/(100 x R) That means if you select V(ILIM_USB)=1V and R = 10 mOhm then I = 1 A * we call it actually MCU_ILIM_USB because that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"
- moved on the sheet: C22, C23, C24, C25, L2, R22, R23, R39, R42, R43, U5
